File: kicad_lna_design/kicad_lna_design.kicad_sch (KiCad schematic)
At the start: 31 parts, among them IC1 SKY67151-396LF, IC2 pga-103+, J1 Conn_Coaxial, J2 Conn_Coaxial, U1 TPS7A4701xRGW

Commit message: updated README
Parts:
- removed L6: 100nH, symbol Device:L
Connections:
- net 13.8V: now reaches C15.2, U1.13 (EN), U1.15 (IN), U1.16 (IN)
Other:
- note added: "LDO auf 5V oder 6V?"
- note added: "abweichungen vom Design Guide PGA-103+: DC-Block von 10nF auf 100pF abgeändert 10nF ist bei 1.3GHz über Resonanz 100pF wirkt für kleinere Frequenzen wie Hochpass RF-Choke von 68nH auf 100nH abgeändert"
- note removed: "abweichungen vom Design Guide PGA-103+: DC-Block von 10nF auf 100pF abgeändert RF-Choke von 68nH auf 100nH abgeändert"
Changed lines of the file:
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@@
 		)
 	)
-	(text "abweichungen vom Design Guide PGA-103+: \nDC-Block von 10nF auf 100pF abgeändert\nRF-Choke von 68nH auf 100nH abgeändert\n"
+	(text "abweichungen vom Design Guide PGA-103+: \nDC-Block von 10nF auf 100pF abgeändert\n		10nF ist bei 1.3GHz über Resonanz\n		100pF wirkt für kleinere Frequenzen wie Hochpass\nRF-Choke von 68nH auf 100nH abgeändert\n\n"
 		(exclude_from_sim no)
-		(at 281.94 197.866 0)
+		(at 243.586 199.39 0)
 		(effects
 			(font
 				(size 1.27 1.27)
 			)
+			(justify left)
 		)
 	)
@@
 		)
 	)
+	(text "LDO auf 5V oder 6V?"
+		(exclude_from_sim no)
+		(at 282.956 217.678 0)
+		(effects
+			(font
+				(size 3.048 3.048)
+			)
+		)
+	)
 	(junction
 		(at 345.44 163.83)
@@
 	)
 	(junction
-		(at 312.42 163.83)
-		(diameter 0)
-		(color 0 0 0 0)
-	)
-	(junction
 		(at 158.75 115.57)
 		(diameter 0)
@@
 	)
 	(junction
-		(at 312.42 142.24)
-		(diameter 0)
-		(color 0 0 0 0)
-	)
-	(junction
 		(at 90.17 142.24)
 		(diameter 0)
@@
 	(junction
 		(at 234.95 142.24)
+		(diameter 0)
+		(color 0 0 0 0)
+	)
+	(junction
+		(at 307.34 163.83)
 		(diameter 0)
 		(color 0 0 0 0)
@@
 	(wire
 		(pts
-			(xy 304.8 142.24) (xy 312.42 142.24)
-		)
-		(stroke
-			(width 0)
-			(type default)
-		)
-	)
-	(wire
-		(pts
 			(xy 102.87 95.25) (xy 102.87 102.87)
 		)
@@
 	(wire
 		(pts
-			(xy 307.34 163.83) (xy 312.42 163.83)
+			(xy 307.34 163.83) (xy 320.04 163.83)
 		)
 		(stroke
@@
 	(wire
 		(pts
+			(xy 298.45 163.83) (xy 307.34 163.83)
+		)
+		(stroke
+			(width 0)
+			(type default)
+		)
+	)
+	(wire
+		(pts
 			(xy 234.95 168.91) (xy 234.95 170.18)
 		)
@@
 	(wire
 		(pts
-			(xy 312.42 163.83) (xy 320.04 163.83)
-		)
-		(stroke
-			(width 0)
-			(type default)
-		)
-	)
-	(wire
-		(pts
 			(xy 325.12 166.37) (xy 320.04 166.37)
 		)
@@
 	(wire
 		(pts
-			(xy 312.42 142.24) (xy 344.17 142.24)
+			(xy 304.8 142.24) (xy 344.17 142.24)
 		)
 		(stroke
@@
 	(wire
 		(pts
-			(xy 312.42 153.67) (xy 312.42 163.83)
-		)
-		(stroke
-			(width 0)
-			(type default)
-		)
-	)
-	(wire
-		(pts
 			(xy 276.86 96.52) (xy 276.86 111.76)
 		)
@@
 		(pts
 			(xy 307.34 172.72) (xy 307.34 173.99)
-		)
-		(stroke
-			(width 0)
-			(type default)
-		)
-	)
-	(wire
-		(pts
-			(xy 312.42 142.24) (xy 312.42 146.05)
 		)
 		(stroke
@@
 				)
 				(justify left)
+				(hide yes)
+			)
+		)
+	)
+	(global_label "13.8V"
+		(shape input)
+		(at 298.45 163.83 180)
+		(fields_autoplaced yes)
+		(effects
+			(font
+				(size 1.27 1.27)
+			)
+			(justify right)
+		)
+		(property "Intersheetrefs" "${INTERSHEET_REFS}"
+			(at 290.1429 163.83 0)
+			(effects
+				(font
+					(size 1.27 1.27)
+				)
+				(justify right)
 				(hide yes)
 			)
@@
 					(unit 1)
 				)
-			)
-		)
-	)
-	(symbol
-		(lib_id "Device:L")
-		(at 312.42 149.86 0)
-		(unit 1)
-		(exclude_from_sim no)
-		(in_bom yes)
-		(on_board yes)
-		(dnp no)
-		(fields_autoplaced yes)
-		(property "Reference" "L6"
-			(at 313.69 148.5899 0)
-			(effects
-				(font
-					(size 1.27 1.27)
-				)
-				(justify left)
-			)
-		)
-		(property "Value" "100nH"
-			(at 313.69 151.1299 0)
-			(effects
-				(font
-					(size 1.27 1.27)
-				)
-				(justify left)
-			)
-		)
-		(property "Footprint" ""
-			(at 312.42 149.86 0)
-			(effects
-				(font
-					(size 1.27 1.27)
-				)
-				(hide yes)
-			)
-		)
-		(property "Datasheet" "~"
-			(at 312.42 149.86 0)
-			(effects
-				(font
-					(size 1.27 1.27)
-				)
-				(hide yes)
-			)
-		)
-		(property "Description" "Inductor"
-			(at 312.42 149.86 0)
-			(effects
-				(font
-					(size 1.27 1.27)
-				)
-				(hide yes)
-			)
-		)
-		(pin "2"
-		)
-		(pin "1"
-		)
-		(instances
-			(project "kicad_lna_design"
-				(path "/64c56d85-b9fa-4642-8dda-836289de401f"
-					(reference "L6")
-					(unit 1)
-				)
